File: udb-s.kicad_sch (KiCad schematic)
At the start: 10 parts, among them J1 TYPE-C-31-M-12, J2 78171-0004, U1 TPD4E05U06DQAR

Commit message: Lil-CC init upload
Parts:
- removed H1: MountingHole, MountingHole:MountingHole_3.2mm_M3_DIN965_Pad_TopBottom, symbol Mechanical:MountingHole_Pad
- removed H2: MountingHole, MountingHole:MountingHole_3.2mm_M3_DIN965_Pad_TopOnly, symbol Mechanical:MountingHole
- removed J2: 78171-0004, locallib:PicoEZMate-Reinforced-Lite, symbol Connector_Generic_MountingPin:Conn_01x04_MountingPin
- added J2, J3: Conn_01x04, acheron_Connectors:Castellated2.54-01x04, symbol Connector_Generic:Conn_01x04
Connections:
- net 5V: now also J2.1 (Pin_1)
- net D+: now also J2.2 (Pin_2)
- net D-: now also J2.3 (Pin_3)
- net GND: now also J2.4 (Pin_4)
- no-connect marks 2 -> 6
Other:
- note added: "Pads"
- note removed: "Pico-EZMate"
